Commit message: 修改xml文件成功

File: tita/urdf/robot.urdf (robot description, URDF)
Before this commit: robot tita, 9 links, 8 joints
Links:
- link base_link: geometry collision box size=0.47 0.3 0.19; visual mesh filename=../meshes/base_link.STL
- link left_leg_1: geometry visual mesh filename=../meshes/left_leg_1.STL
- link left_leg_2: geometry visual mesh filename=../meshes/left_leg_2.STL
- link left_leg_3: geometry collision box size=0.2 0.07 0.05; visual mesh filename=../meshes/left_leg_3.STL
- link left_leg_4: geometry collision cylinder length=0.034 radius=0.0925; visual mesh filename=../meshes/left_leg_4.STL
- link right_leg_1: geometry visual mesh filename=../meshes/right_leg_1.STL
- link right_leg_2: geometry visual mesh filename=../meshes/right_leg_2.STL
- link right_leg_3: geometry collision box size=0.2 0.07 0.05; visual mesh filename=../meshes/right_leg_3.STL
- link right_leg_4: geometry collision cylinder length=0.034 radius=0.0925; visual mesh filename=../meshes/right_leg_4.STL
