Commit message: 修改模型

File: tita/urdf/robot_backup.urdf (robot description, URDF)
Before this commit: robot tita, 9 links, 8 joints
Links:
- added link ch201
- added link imu_link, mass 0.001; collision box size=.001 .001 .001; visual box size=0.001 0.001 0.001
- added link left_camera
- added link right_camara
- added link spad
- added link spad1
Joints:
- added joint ch201: type fixed, parent base_link, child ch201, origin xyz=0.23782 0 0.018636 rpy=1.1693 0 1.5708, axis 0 0 0
- added joint imu_joint: type fixed, parent base_link, child imu_link, origin xyz=0 0 0 rpy=0 0 0
- added joint left_camera: type fixed, parent base_link, child left_camera, origin xyz=0.23416 0.075 0.04036 rpy=1.5708 0 1.5708, axis 0 0 0
- added joint right_camera: type fixed, parent base_link, child right_camara, origin xyz=0.23416 -0.075001 0.04036 rpy=1.5708 0 1.5708, axis 0 0 0
- added joint spad: type fixed, parent base_link, child spad, origin xyz=0.24052 -0.0019 0.064455 rpy=2.199 0 1.5708, axis 0 0 0
- added joint spad1: type fixed, parent base_link, child spad1, origin xyz=0.21953 -0.0019 -0.030142 rpy=2.632 0 1.5708, axis 0 0 0

Commit message: 完成mjcf模型

File: tita/urdf/robot_backup.urdf (robot description, URDF)
Before this commit: robot tita, 15 links, 14 joints
Links:
- link base_link: geometry collision box size=0.47 0.3 0.19; visual mesh filename=../meshes/base_link.STL
- link left_leg_1: geometry visual mesh filename=../meshes/left_leg_1.STL
- link left_leg_2: geometry visual mesh filename=../meshes/left_leg_2.STL
- link left_leg_3: geometry collision box size=0.2 0.07 0.05; visual mesh filename=../meshes/left_leg_3.STL
- link left_leg_4: geometry collision cylinder length=0.034 radius=0.0925; visual mesh filename=../meshes/left_leg_4.STL
- link right_leg_1: geometry visual mesh filename=../meshes/right_leg_1.STL
- link right_leg_2: geometry visual mesh filename=../meshes/right_leg_2.STL
- link right_leg_3: geometry collision box size=0.2 0.07 0.05; visual mesh filename=../meshes/right_leg_3.STL
- link right_leg_4: geometry collision cylinder length=0.034 radius=0.0925; visual mesh filename=../meshes/right_leg_4.STL

File: tita/urdf/robot_with_tower.urdf (robot description, URDF)
Before this commit: robot tita, 17 links, 16 joints
Links:
- link base_link: geometry collision box size=0.47 0.3 0.19; visual mesh filename=../meshes/base_link.STL
- link left_leg_1: geometry visual mesh filename=../meshes/left_leg_1.STL
- link left_leg_2: geometry visual mesh filename=../meshes/left_leg_2.STL
- link left_leg_3: geometry collision box size=0.2 0.07 0.05; visual mesh filename=../meshes/left_leg_3.STL
- link left_leg_4: geometry collision cylinder length=0.034 radius=0.0925; visual mesh filename=../meshes/left_leg_4.STL
- link radar_link: geometry visual mesh filename=../../tower/meshes/radar_link.STL
- link right_leg_1: geometry visual mesh filename=../meshes/right_leg_1.STL
- link right_leg_2: geometry visual mesh filename=../meshes/right_leg_2.STL
- link right_leg_3: geometry collision box size=0.2 0.07 0.05; visual mesh filename=../meshes/right_leg_3.STL
- link right_leg_4: geometry collision cylinder length=0.034 radius=0.0925; visual mesh filename=../meshes/right_leg_4.STL
- link tower_base_link: geometry collision box size=0.132 0.132 0.180; visual mesh filename=../../tower/meshes/base_link.STL
